File: PCB/halloween_badge/halloween_badge.kicad_sch (KiCad schematic)
At the start: 20 parts, among them SW1 SW_SPDT, U1 ATtiny48-A

Commit message: first finished PCB design
Parts:
- added D5: LED_Filled, LED_SMD:LED_0603_1608Metric_Pad1.05x0.95mm_HandSolder, symbol Device:LED_Filled
- added R6: R, Resistor_SMD:R_0402_1005Metric_Pad0.72x0.64mm_HandSolder, symbol Device:R
- BT1: footprint Battery:BatteryHolder_Keystone_3002_1x2032 -> Connector_PinHeader_2.54mm:PinHeader_2x01_P2.54mm_Vertical_SMD
- C1, C2: footprint Capacitor_SMD:C_0805_2012Metric_Pad1.18x1.45mm_HandSolder -> Capacitor_SMD:C_0402_1005Metric_Pad0.74x0.62mm_HandSolder
- R1, R2, R3, R4, R5: footprint Resistor_SMD:R_0805_2012Metric_Pad1.20x1.40mm_HandSolder -> Resistor_SMD:R_0402_1005Metric_Pad0.72x0.64mm_HandSolder
- SW1: footprint (none) -> Button_Switch_SMD:SW_SPDT_CK_JS102011SAQN
Connections:
- net GND: now also D5.1 (K)
- net led_eye_left: now also U1.24 (PC1)
- net led_eye_right: now also U1.28 (PC5)
- net led_mouth_left: now also U1.25 (PC2)
- net led_mouth_right: now also U1.27 (PC4)
- net led_nose: now reaches U1.26 (PC3)
- net led_nose: now also R6.1
- new net: D5.2 (A), R6.2
Other:
- moved on the sheet: R1, TP1
